File: Parts/SteeringWheel2025/steering_pcb/steering_pcb.kicad_pcb (KiCad board)
At the start: 2 copper layers, 102 x 102 mm, 189 parts, among them J0 Quick_connector, J1 Button 1 molex-µfit connector, J10 Button 1 molex-µfit connector, J11 Button 1 molex-µfit connector, J12 Button 1 molex-µfit connector, J13 PINHD_1x1_Male, J15 CAN pin header, J2 Button 1 molex-µfit connector, J3 Button 1 molex-µfit connector, J4 Button 1 molex-µfit connector, J5 Button 1 molex-µfit connector, J6 Button 1 molex-µfit connector, J7 Button 1 molex-µfit connector, J8 Button 1 molex-µfit connector, J9 Button 1 molex-µfit connector, Q1 BSS138BKS, Q10 2N7002DW, Q11 2N7002DW, Q12 2N7002DW, Q13 2N7002DW, Q14 2N7002DW, Q15 2N7002DW, Q16 2N7002DW, Q17 2N7002DW, Q18 2N7002DW, Q19 2N7002DW, Q2 2N7002DW, Q20 2N7002DW, Q21 2N7002DW, Q3 2N7002DW, Q4 BS170, Q5 2N7002DW, Q6 BSS138BKS, Q7 2N7002DW, Q8 2N7002DW, Q9 2N7002DW, SW1 Push_Button, U1 MCP2515-xSO, U2 TPS5430DDA, U3 TPS5430DDA, U5 ISM330DHCX, U6 TJA1051T-3, Y1 16MHz

Commit message: pcb backup
Parts:
- JP1, JP6, Q1, Q6, R10, R12, R13, R8, R9, U5: moved to F.Cu
- TP_SCL3v1, TP_SDA3v1: moved to B.Cu
- moved R53 383.1 mm to (132.3, 48.4)
- moved R56 383.1 mm to (132.3, 58.7)
- moved R59 383.1 mm to (132.3, 56.2)
- moved D8 383.1 mm to (139.7, 58.2)
- moved DZ8 383.1 mm to (143.0, 58.2)
- moved Q14 383.1 mm to (134.5, 58.6)
- moved Q15 383.1 mm to (137.3, 54.6)
- moved R55 383.1 mm to (134.3, 47.9)
- moved R57 383.1 mm to (141.7, 60.2)
- moved R60 383.1 mm to (143.5, 45.1)
- moved J8 383.1 mm to (149.1, 53.7)
- moved R50 383.1 mm to (137.4, 49.1)
- moved R58 383.1 mm to (149.4, 45.6)
- moved R61 383.1 mm to (134.9, 54.1)
- moved R54 341.7 mm to (173.4, 46.4), turned to 0 degrees
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Routing:
- net +3.3V: track 123.6 -> 105.0 mm, vias 3 -> 5
- net /LED and Buttons/Connector_4/button_1_1: track 11.3 -> 3.52 mm
- net /LED and Buttons/Connector_4/button_1_2: track 11.8 -> 4.61 mm
- net SCL_3V: track 12.1 -> 5.05 mm, vias 2 -> 1
- net /LED and Buttons/Connector_4/button_1_0: track 12.1 -> 5.60 mm
- net SDO: track 6.88 -> 2.78 mm
- net SDA_3V: track 4.50 -> 8.06 mm, vias 0 -> 1
- net Net-(DZ7C-C3): track 6.43 -> 9.62 mm
- net MCU_SDA: track 7.34 -> 4.45 mm
- net MCU_SCL: track 7.22 -> 4.78 mm
- net Net-(Q13B-D2): track 1.80 -> 4.14 mm
- net /LED and Buttons/Connector_4/button_1_3: track 14.7 -> 12.4 mm
- net Net-(JP6-A): track 17.2 -> 18.5 mm
- net button2_0: track 58.8 -> 59.5 mm
- net Net-(A1-D0/RX0): track 16.4 -> 17.1 mm
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