File: Parts/steering_wheel_2025/steering_pcb/CAN_BUS.kicad_sch (KiCad schematic)
At the start: 20 parts, among them U1 MCP2515-xSO, U6 TJA1051T-3, Y1 16MHz

Commit message: Dashboard electron
Parts:
- added C18: 0.1uF, Capacitor_SMD:C_0805_2012Metric_Pad1.18x1.45mm_HandSolder, symbol Device:C_Small
- added C20, C21: 14pF, Capacitor_SMD:C_0805_2012Metric_Pad1.18x1.45mm_HandSolder, symbol Device:C_Small
- added C22: 4700pF, Capacitor_SMD:C_0805_2012Metric_Pad1.18x1.45mm_HandSolder, symbol Device:C_Small
- added D18: PESD1CAN, PCM_Package_TO_SOT_SMD_AKL:SOT-23, symbol PCM_Diode_TVS_AKL:PESD1CAN
- added JP2, JP7: ~, Jumper:SolderJumper-2_P1.3mm_Bridged_RoundedPad1.0x1.5mm, symbol Jumper:SolderJumper_2_Bridged
- added R90: 120, Resistor_SMD:R_0402_1005Metric_Pad0.72x0.64mm_HandSolder, symbol Device:R_Small
- added R91, R92: 60, Resistor_SMD:R_0402_1005Metric_Pad0.72x0.64mm_HandSolder, symbol Device:R_Small
- added R93: 300, Resistor_SMD:R_0402_1005Metric_Pad0.72x0.64mm_HandSolder, symbol Device:R_Small
- added U4: MCP2561FD-H-SN, Package_SO:SOIC-8-1EP_3.9x4.9mm_P1.27mm_EP2.29x3mm, symbol Steering_Wheel_project:MCP2561FD-H-SN
- C1, C2: value 15pF -> 14pF
Connections:
- net +5V_MCU: now also JP2.2 (B)
- net CAN_H: now also D18.1 (A1), R91.1, U4.7 (CANH)
- net CAN_L: now also D18.2 (A2), R92.2, U4.6 (CANL)
- net GND: now also C18.2, C20.2, C22.1, D18.3 (Com), U4.2 (VSS)
- new net: C21.1, JP7.2 (B)
- new net: C20.1, C21.2, R90.2
- new net: C18.1, JP2.1 (A), U4.3 (VDD)
- new net: R93.1, U4.5 (SPLIT)
- new net: C22.2, R91.2, R92.1, R93.2
- new net: JP7.1 (A), R90.1
- new net CAN_RX: U4.4 (RXD)
- new net CAN_STBY: U4.8 (STBY)
- new net CAN_TX: U4.1 (TXD)
Other:
- note added: "Is better to use 2561fd + ESD + crystal"
- note added: "Optional resistor to allow communication during bus failure (CANL shorted to ground)."
- note removed: "Inspiration from: https://learn.adafruit.com/adafruit-can-pal https://learn.adafruit.com/adafruit-can-bus-featherwing https://learn.adafruit.com/adafruit-feather-m4-express-atsamd51"
- moved on the sheet: C1, C12, C13, C14, C15, C2, C4, D14, D16, D17, JP3, JP4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
