File: Parts/steering_wheel_2025/steering_pcb/CAN_BUS.kicad_sch (KiCad schematic)
At the start: 20 parts, among them U1 MCP2515-xSO, U6 TJA1051T-3, Y1 16MHz

Commit message: slight changes in schematic
Parts:
- R2: symbol Device:R -> Device:R_Small
Changed lines of the file:
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@@
 	(wire
 		(pts
+			(xy 167.64 58.42) (xy 167.64 59.69)
+		)
+		(stroke
+			(width 0)
+			(type default)
+		)
+	)
+	(wire
+		(pts
 			(xy 107.95 69.85) (xy 105.41 69.85)
 		)
@@
 	(wire
 		(pts
+			(xy 167.64 64.77) (xy 167.64 66.04)
+		)
+		(stroke
+			(width 0)
+			(type default)
+		)
+	)
+	(wire
+		(pts
 			(xy 123.19 31.75) (xy 123.19 34.29)
 		)
@@
 	)
 	(symbol
-		(lib_id "Device:R")
+		(lib_id "Device:R_Small")
 		(at 167.64 62.23 0)
 		(unit 1)
@@
 		)
 		(property "Footprint" "Resistor_SMD:R_0402_1005Metric_Pad0.72x0.64mm_HandSolder"
-			(at 165.862 62.23 90)
+			(at 167.64 62.23 0)
 			(effects
 				(font
@@
 			)
 		)
-		(property "Datasheet" "https://www.lcsc.com/datasheet/lcsc_datasheet_2205311845_UNI-ROYAL-Uniroyal-Elec-0402WGJ0103TCE_C25531.pdf"
+		(property "Datasheet" "~"
 			(at 167.64 62.23 0)
 			(effects
@@
 			)
 		)
-		(property "Description" "Resistor"
+		(property "Description" "Resistor, small symbol"
 			(at 167.64 62.23 0)
 			(effects

Commit message: Error fixing with kicad_dru, and silkscreeen updates. TO-DO: BOM to basic
Parts:
- JP3, JP4: now not fitted
- JP5: Note (none) -> CAN power connection; now not fitted
- R1, R2, R26, R3, Y1: Note (none) -> basic
Changed lines of the file:
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@@
 		(in_bom no)
 		(on_board yes)
-		(dnp no)
+		(dnp yes)
 		(property "Reference" "JP3"
 			(at 151.13 78.994 0)
@@
 			)
 		)
-		(property "Description" "Resistor, small symbol"
+		(property "Description" "0402WGF1001TCE"
 			(at 154.94 35.56 0)
 			(effects
@@
 		)
 		(property "Rating" ""
+			(at 154.94 35.56 0)
+			(effects
+				(font
+					(size 1.27 1.27)
+				)
+				(hide yes)
+			)
+		)
+		(property "Note" "basic"
 			(at 154.94 35.56 0)
 			(effects
@@
 			)
 		)
-		(property "Description" "Four pin 16MHz crystal, GND on pins 2 and 4, small symbol"
+		(property "Description" "X322516MLB4SI"
 			(at 102.87 69.85 0)
 			(effects
@@
 		)
 		(property "Rating" ""
+			(at 102.87 69.85 0)
+			(effects
+				(font
+					(size 1.27 1.27)
+				)
+				(hide yes)
+			)
+		)
+		(property "Note" "basic"
 			(at 102.87 69.85 0)
 			(effects
@@
 			)
 		)
-		(property "Description" "Resistor, small symbol"
+		(property "Description" "0402WGF1001TCE"
 			(at 147.32 35.56 0)
 			(effects
@@
 			)
 		)
+		(property "Note" "basic"
+			(at 147.32 35.56 0)
+			(effects
+				(font
+					(size 1.27 1.27)
+				)
+				(hide yes)
+			)
+		)
 		(pin "1"
 		)
@@
 		(in_bom no)
 		(on_board yes)
-		(dnp no)
+		(dnp yes)
 		(property "Reference" "JP5"
 			(at 143.764 27.94 0)
@@
 		)
 		(property "Rating" ""
+			(at 140.97 27.94 0)
+			(effects
+				(font
+					(size 1.27 1.27)
+				)
+				(hide yes)
+			)
+		)
+		(property "Note" "CAN power connection"
 			(at 140.97 27.94 0)
 			(effects
@@
 			)
 		)
-		(property "Datasheet" "~"
+		(property "Datasheet" "https://jlcpcb.com/partdetail/C25531"
 			(at 167.64 62.23 0)
 			(effects
@@
 			)
 		)
-		(property "Description" "Resistor, small symbol"
+		(property "Description" "0402WGJ0103TCE"
 			(at 167.64 62.23 0)
 			(effects
@@
 		)
 		(property "Rating" ""
+			(at 167.64 62.23 0)
+			(effects
+				(font
+					(size 1.27 1.27)
+				)
+				(hide yes)
+			)
+		)
+		(property "Note" "basic"
 			(at 167.64 62.23 0)
 			(effects
@@
 			)
 		)
-		(property "Description" "Resistor, small symbol"
+		(property "Description" "0402WGF1200TCE"
 			(at 200.66 55.88 0)
 			(effects
@@
 			)
 		)
+		(property "Note" "basic"
+			(at 200.66 55.88 0)
+			(effects
+				(font
+					(size 1.27 1.27)
+				)
+				(hide yes)
+			)
+		)
 		(pin "1"
 		)
@@
 		(in_bom no)
 		(on_board yes)
-		(dnp no)
+		(dnp yes)
 		(property "Reference" "JP4"
 			(at 203.2 48.2599 90)

Commit message: board update
Parts:
- added C18, C19, C20: 20pF, Capacitor_SMD:C_0805_2012Metric_Pad1.18x1.45mm_HandSolder, symbol Device:C_Small
- C1, C2: value 15pF -> 20pF; JLCPCB C63339 -> C1798; Note (none) -> basic; Product (none) -> CL21C200JBANNNC
- C12, C14, C15: Product (none) -> 0805CG150J500NT; now not fitted; now left out of the parts list
- C13, C4: JLCPCB C126469 -> C49678; Note (none) -> basic; Product (none) -> YAGEO-CC0805KRX7R9BB104
- D14: value PESD1CAN -> ~; footprint PCM_Package_TO_SOT_SMD_AKL:SOT-23 -> Package_TO_SOT_SMD:SOT-23; Note (none) -> no; Product (none) -> PESD1CAN
- D16, D17: value KT-0603R -> ~; Note (none) -> basic; Product (none) -> KT-0603R
- R1, R3: Product (none) -> 0402WGF1001TCE
- R2: Product (none) -> 0402WGJ0103TCE
- R26: Product (none) -> 0402WGF1200TCE
- U1, U6: Note (none) -> no
- Y1: Product (none) -> X322516MLB4SI
Connections:
- net CAN_H: now also C18.2, C19.1; no longer C12.1, C15.1
- net CAN_L: now also C18.1, C20.2; no longer C12.2, C14.1
- net GND: now also C19.2, C20.1; no longer C14.2, C15.2
Other:
- note added: "caps were replaced with cheaper 20pF versions"

Commit message: Rename folders for consistency
Parts:
- D14: value ~ -> PESD1CAN
- D16, D17: value ~ -> KT-0603R
- R1, R3: value 1k -> 1kΩ
- R2: value 10k -> 10kΩ
- R26: value 120 -> 120Ω
Changed lines of the file:
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@@
 (kicad_sch
-	(version 20231120)
+	(version 20250114)
 	(generator "eeschema")
-	(generator_version "8.0")
+	(generator_version "9.0")
 	(paper "A4")
 	(title_block
@@
 		(company "DTU ROAST")
 	)
+	(rectangle
+		(start 177.8 87.63)
+		(end 236.22 99.06)
+		(stroke
+			(width 0)
+			(type default)
+		)
+		(fill
+			(type none)
+		)
+	)
+	(rectangle
+		(start 87.63 18.542)
+		(end 247.65 85.09)
+		(stroke
+			(width 0)
+			(type default)
+		)
+		(fill
+			(type none)
+		)
+	)
+	(text "caps were replaced\nwith cheaper 20pF\nversions"
+		(exclude_from_sim no)
+		(at 213.36 92.71 0)
+		(effects
+			(font
+				(size 1.27 1.27)
+			)
+			(justify left)
+		)
+	)
+	(text "Inspiration from:\nhttps://learn.adafruit.com/adafruit-can-pal\nhttps://learn.adafruit.com/adafruit-can-bus-featherwing\nhttps://learn.adafruit.com/adafruit-feather-m4-express-atsamd51"
+		(exclude_from_sim no)
+		(at 177.292 171.45 0)
+		(effects
+			(font
+				(size 1.27 1.27)
+			)
+			(justify left)
+		)
+	)
+	(text "CAN transceiver and a controller"
+		(exclude_from_sim no)
+		(at 89.916 25.146 0)
+		(effects
+			(font
+				(size 0.9 0.9)
+			)
+			(justify left)
+		)
+	)
+	(text "CAN"
+		(exclude_from_sim no)
+		(at 92.71 22.606 0)
+		(effects
+			(font
+				(size 2 2)
+				(thickness 0.4)
+				(bold yes)
+			)
+		)
+	)
 	(junction
 		(at 154.94 31.75)
@@
 		)
 	)
-	(rectangle
-		(start 177.8 87.63)
-		(end 236.22 99.06)
-		(stroke
-			(width 0)
-			(type default)
-		)
-		(fill
-			(type none)
-		)
-	)
-	(rectangle
-		(start 87.63 18.542)
-		(end 247.65 85.09)
-		(stroke
-			(width 0)
-			(type default)
-		)
-		(fill
-			(type none)
-		)
-	)
 	(image
 		(at 78.74 167.64)
@@
 		)
 	)
-	(text "caps were replaced\nwith cheaper 20pF\nversions"
-		(exclude_from_sim no)
-		(at 213.36 92.71 0)
-		(effects
-			(font
-				(size 1.27 1.27)
-			)
-			(justify left)
-		)
-	)
-	(text "Inspiration from:\nhttps://learn.adafruit.com/adafruit-can-pal\nhttps://learn.adafruit.com/adafruit-can-bus-featherwing\nhttps://learn.adafruit.com/adafruit-feather-m4-express-atsamd51"
-		(exclude_from_sim no)
-		(at 177.292 171.45 0)
-		(effects
-			(font
-				(size 1.27 1.27)
-			)
-			(justify left)
-		)
-	)
-	(text "CAN transceiver and a controller"
-		(exclude_from_sim no)
-		(at 89.916 25.146 0)
-		(effects
-			(font
-				(size 0.9 0.9)
-			)
-			(justify left)
-		)
-	)
-	(text "CAN"
-		(exclude_from_sim no)
-		(at 92.71 22.606 0)
-		(effects
-			(font
-				(size 2 2)
-				(thickness 0.4)
-				(bold yes)
-			)
-		)
-	)
 	(global_label "CAN_L"
 		(shape input)
@@
 			)
 		)
-		(property "Value" "~"
+		(property "Value" "KT-0603R"
 			(at 156.718 40.894 90)
 			(effects
@@
 			)
 		)
-		(property "Value" "~"
+		(property "Value" "KT-0603R"
 			(at 145.542 40.894 90)
 			(effects
@@
 			)
 		)
-		(property "Value" "1k"
+		(property "Value" "1kΩ"
 			(at 159.004 36.576 0)
 			(effects
@@
 			)
 		)
-		(property "Value" "~"
+		(property "Value" "PESD1CAN"
 			(at 234.95 49.276 0)
 			(effects
@@
 			)
 		)
-		(property "Value" "1k"
+		(property "Value" "1kΩ"
 			(at 151.13 36.576 0)
 			(effects
@@
 			)
 		)
-		(property "Value" "10k"
+		(property "Value" "10kΩ"
 			(at 166.37 63.5 0)
 			(effects
@@
 			)
 		)
-		(property "Value" "120"
+		(property "Value" "120Ω"
 			(at 201.93 56.896 0)
 			(effects
