File: Parts/steering_wheel_2025/steering_pcb/conn_1-2.kicad_sch (KiCad schematic)
At the start: 21 parts, among them J1 Button 1 molex-µfit connector, J2 Button 1 molex-µfit connector, Q2 2N7002DW, Q3 2N7002DW, Q5 2N7002DW

Commit message: Dashboard electron
Parts:
- J1, J2: now fitted
Other:
- moved on the sheet: D1A, D1B, D1C, D2A, D2B, D2C, DZ1A, DZ1B, DZ1C, DZ2A, DZ2B, DZ2C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
