File: Parts/steering_wheel_2025/steering_pcb/gyroschope.kicad_sch (KiCad schematic)
At the start: 12 parts, among them Q1 BSS138BKS, Q6 BSS138BKS, U5 ISM330DHCX

Commit message: slight changes in schematic
Parts:
- R10, R12, R13, R9: symbol Device:R -> Device:R_Small
Other:
- note added: "Alternative power supply, but currently power is delivered by the 3v3 directly from the arduino MCU"
Changed lines of the file:
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@@
+	(wire
+		(pts
+			(xy 215.9 54.61) (xy 215.9 59.69)
+		)
+		(stroke
+			(width 0)
+			(type default)
+		)
+	)
+	(wire
+		(pts
+			(xy 193.04 54.61) (xy 193.04 59.69)
+		)
+		(stroke
+			(width 0)
+			(type default)
+		)
+	)
 	(wire
 		(pts
@@
 	(wire
 		(pts
-			(xy 162.56 58.42) (xy 162.56 59.69)
-		)
-		(stroke
-			(width 0)
-			(type default)
-		)
-	)
-	(wire
-		(pts
-			(xy 193.04 55.88) (xy 193.04 59.69)
+			(xy 193.04 45.72) (xy 193.04 49.53)
+		)
+		(stroke
+			(width 0)
+			(type default)
+		)
+	)
+	(wire
+		(pts
+			(xy 162.56 50.8) (xy 162.56 52.07)
 		)
 		(stroke
@@
 	(wire
 		(pts
-			(xy 215.9 55.88) (xy 215.9 59.69)
+			(xy 139.7 54.61) (xy 139.7 59.69)
+		)
+		(stroke
+			(width 0)
+			(type default)
+		)
+	)
+	(wire
+		(pts
+			(xy 215.9 48.26) (xy 215.9 49.53)
 		)
 		(stroke
@@
 	(wire
 		(pts
-			(xy 193.04 45.72) (xy 193.04 48.26)
-		)
-		(stroke
-			(width 0)
-			(type default)
-		)
-	)
-	(wire
-		(pts
 			(xy 139.7 59.69) (xy 134.62 59.69)
 		)
@@
 	(wire
 		(pts
-			(xy 139.7 45.72) (xy 139.7 48.26)
-		)
-		(stroke
-			(width 0)
-			(type default)
-		)
-	)
-	(wire
-		(pts
-			(xy 139.7 55.88) (xy 139.7 59.69)
+			(xy 139.7 45.72) (xy 139.7 49.53)
 		)
 		(stroke
@@
 		(pts
 			(xy 139.7 59.69) (xy 146.05 59.69)
+		)
+		(stroke
+			(width 0)
+			(type default)
+		)
+	)
+	(wire
+		(pts
+			(xy 162.56 57.15) (xy 162.56 59.69)
 		)
 		(stroke
@@
 	)
 	(image
-		(at 155.956 137.414)
+		(at 220.726 142.494)
 		(scale 0.397734)
 		(data "iVBORw0KGgoAAAANSUhEUgAAAwQAAAFUCAIAAAAViGxrAAAACXBIWXMAAA7EAAAOxAGVKw4bAAAX"
@@
 		)
 	)
+	(text "Alternative power supply, but currently power is delivered by the 3v3 directly from the arduino MCU"
+		(exclude_from_sim no)
+		(at 224.028 125.476 0)
+		(effects
+			(font
+				(size 1.27 1.27)
+			)
+		)
+	)
 	(text "I2C Address pin. Pulling this pin high or bridging\nthe solder jumper on the back will change the I2C\naddress from 0x6A to 0x6B"
 		(exclude_from_sim no)
@@
 	)
 	(symbol
-		(lib_id "Device:R")
+		(lib_id "Device:R_Small")
 		(at 162.56 54.61 0)
 		(unit 1)
@@
 		)
 		(property "Footprint" "Resistor_SMD:R_0402_1005Metric_Pad0.72x0.64mm_HandSolder"
-			(at 160.782 54.61 90)
-			(effects
-				(font
-					(size 1.27 1.27)
-				)
-				(hide yes)
-			)
-		)
-		(property "Datasheet" "https://www.lcsc.com/datasheet/lcsc_datasheet_2205311845_UNI-ROYAL-Uniroyal-Elec-0402WGJ0103TCE_C25531.pdf"
 			(at 162.56 54.61 0)
 			(effects
@@
 			)
 		)
-		(property "Description" "Resistor"
+		(property "Datasheet" "~"
+			(at 162.56 54.61 0)
+			(effects
+				(font
+					(size 1.27 1.27)
+				)
+				(hide yes)
+			)
+		)
+		(property "Description" "Resistor, small symbol"
 			(at 162.56 54.61 0)
 			(effects
@@
 	)
 	(symbol
-		(lib_id "Device:R")
+		(lib_id "Device:R_Small")
 		(at 193.04 52.07 0)
 		(unit 1)
@@
 		)
 		(property "Footprint" "Resistor_SMD:R_0402_1005Metric_Pad0.72x0.64mm_HandSolder"
-			(at 191.262 52.07 90)
-			(effects
-				(font
-					(size 1.27 1.27)
-				)
-				(hide yes)
-			)
-		)
-		(property "Datasheet" "https://www.lcsc.com/datasheet/lcsc_datasheet_2205311845_UNI-ROYAL-Uniroyal-Elec-0402WGJ0103TCE_C25531.pdf"
 			(at 193.04 52.07 0)
 			(effects
@@
 			)
 		)
-		(property "Description" "Resistor"
+		(property "Datasheet" "~"
+			(at 193.04 52.07 0)
+			(effects
+				(font
+					(size 1.27 1.27)
+				)
+				(hide yes)
+			)
+		)
+		(property "Description" "Resistor, small symbol"
 			(at 193.04 52.07 0)
 			(effects
@@
 	)
 	(symbol
-		(lib_id "Device:R")
+		(lib_id "Device:R_Small")
 		(at 139.7 52.07 0)
 		(unit 1)
@@
 		)
 		(property "Footprint" "Resistor_SMD:R_0402_1005Metric_Pad0.72x0.64mm_HandSolder"
-			(at 137.922 52.07 90)
-			(effects
-				(font
-					(size 1.27 1.27)
-				)
-				(hide yes)
-			)
-		)
-		(property "Datasheet" "https://www.lcsc.com/datasheet/lcsc_datasheet_2205311845_UNI-ROYAL-Uniroyal-Elec-0402WGJ0103TCE_C25531.pdf"
 			(at 139.7 52.07 0)
 			(effects
@@
 			)
 		)
-		(property "Description" "Resistor"
+		(property "Datasheet" "~"
+			(at 139.7 52.07 0)
+			(effects
+				(font
+					(size 1.27 1.27)
+				)
+				(hide yes)
+			)
+		)
+		(property "Description" "Resistor, small symbol"
 			(at 139.7 52.07 0)
 			(effects
@@
 	)
 	(symbol
-		(lib_id "Device:R")
+		(lib_id "Device:R_Small")
 		(at 215.9 52.07 0)
 		(unit 1)
@@
 		)
 		(property "Footprint" "Resistor_SMD:R_0402_1005Metric_Pad0.72x0.64mm_HandSolder"
-			(at 214.122 52.07 90)
-			(effects
-				(font
-					(size 1.27 1.27)
-				)
-				(hide yes)
-			)
-		)
-		(property "Datasheet" "https://www.lcsc.com/datasheet/lcsc_datasheet_2205311845_UNI-ROYAL-Uniroyal-Elec-0402WGJ0103TCE_C25531.pdf"
 			(at 215.9 52.07 0)
 			(effects
@@
 			)
 		)
-		(property "Description" "Resistor"
+		(property "Datasheet" "~"
 			(at 215.9 52.07 0)
 			(effects
+				(font
+					(size 1.27 1.27)
+				)
+				(hide yes)
+			)
+		)
+		(property "Description" "Resistor, small symbol"
+			(at 215.9 52.07 0)
+			(effects

Commit message: Dashboard electron
Other:
- note added: "I2C pullup and shift"
- note removed: "Reference: https://learn.adafruit.com/lsm6dsox-and-ism330dhc-6-dof-imu?view=all credits to adafruit"
- note removed: "i2c pullup and shift"
- moved on the sheet: JP1, JP6, Q1A, Q6A, R10, R12, R13, R8, R9, TP_SCL3v1, TP_SDA3v1, U5
