File: Parts/steering_wheel_2025/steering_pcb/gyroschope.kicad_sch (KiCad schematic)
At the start: 12 parts, among them Q1 BSS138BKS, Q6 BSS138BKS, U5 ISM330DHCX

Commit message: Error fixing with kicad_dru, and silkscreeen updates. TO-DO: BOM to basic
Parts:
- JP1: Note (none) -> I2C address pin; now not fitted
- JP6: Note (none) -> Gyroscope power solder jumper; now not fitted
- R10, R12, R13, R8, R9: Note (none) -> basic
Connections:
- net +5V renamed +5V_MCU
Changed lines of the file:
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@@
 			)
 		)
-		(property "Datasheet" "~"
+		(property "Datasheet" "https://jlcpcb.com/partdetail/C25531"
 			(at 162.56 54.61 0)
 			(effects
@@
 			)
 		)
-		(property "Description" "Resistor, small symbol"
+		(property "Description" "0402WGJ0103TCE"
 			(at 162.56 54.61 0)
 			(effects
@@
 		)
 		(property "Rating" ""
+			(at 162.56 54.61 0)
+			(effects
+				(font
+					(size 1.27 1.27)
+				)
+				(hide yes)
+			)
+		)
+		(property "Note" "basic"
 			(at 162.56 54.61 0)
 			(effects
@@
 	)
 	(symbol
-		(lib_id "power:+5V")
-		(at 215.9 48.26 0)
+		(lib_id "power:+12V")
+		(at 162.56 50.8 0)
 		(unit 1)
 		(exclude_from_sim no)
@@
 		(on_board yes)
 		(dnp no)
-		(fields_autoplaced yes)
-		(property "Reference" "#PWR042"
-			(at 215.9 52.07 0)
-			(effects
-				(font
-					(size 1.27 1.27)
-				)
-				(hide yes)
-			)
-		)
-		(property "Value" "+5V"
-			(at 215.9 43.18 0)
-			(effects
-				(font
-					(size 1.27 1.27)
+		(property "Reference" "#PWR38"
+			(at 162.56 54.61 0)
+			(effects
+				(font
+					(size 1.27 1.27)
+				)
+				(hide yes)
+			)
+		)
+		(property "Value" "+5V_MCU"
+			(at 162.56 46.736 0)
+			(effects
+				(font
+					(size 0.635 0.635)
 				)
 			)
 		)
 		(property "Footprint" ""
-			(at 215.9 48.26 0)
+			(at 162.56 50.8 0)
 			(effects
 				(font
@@
 		)
 		(property "Datasheet" ""
-			(at 215.9 48.26 0)
-			(effects
-				(font
-					(size 1.27 1.27)
-				)
-				(hide yes)
-			)
-		)
-		(property "Description" "Power symbol creates a global label with name \"+5V\""
-			(at 215.9 48.26 0)
+			(at 162.56 50.8 0)
+			(effects
+				(font
+					(size 1.27 1.27)
+				)
+				(hide yes)
+			)
+		)
+		(property "Description" ""
+			(at 162.56 50.8 0)
 			(effects
 				(font
@@
 			(project "steering_pcb"
 				(path "/27c2abcd-4c9d-416a-9e0c-4ab4decfd0fd/3158a1dc-35f2-49d2-93b5-e8517c53d7ab"
-					(reference "#PWR042")
+					(reference "#PWR38")
 					(unit 1)
 				)
@@
 			)
 		)
-		(property "Datasheet" "~"
+		(property "Datasheet" "https://jlcpcb.com/partdetail/C25531"
 			(at 193.04 52.07 0)
 			(effects
@@
 			)
 		)
-		(property "Description" "Resistor, small symbol"
+		(property "Description" "0402WGJ0103TCE"
 			(at 193.04 52.07 0)
 			(effects
@@
 		)
 		(property "Rating" ""
+			(at 193.04 52.07 0)
+			(effects
+				(font
+					(size 1.27 1.27)
+				)
+				(hide yes)
+			)
+		)
+		(property "Note" "basic"
 			(at 193.04 52.07 0)
 			(effects
@@
 			)
 		)
-		(property "Datasheet" "~"
+		(property "Datasheet" "https://jlcpcb.com/partdetail/C25531"
 			(at 139.7 52.07 0)
 			(effects
@@
 			)
 		)
-		(property "Description" "Resistor, small symbol"
+		(property "Description" "0402WGJ0103TCE"
 			(at 139.7 52.07 0)
 			(effects
@@
 		)
 		(property "Rating" ""
+			(at 139.7 52.07 0)
+			(effects
+				(font
+					(size 1.27 1.27)
+				)
+				(hide yes)
+			)
+		)
+		(property "Note" "basic"
 			(at 139.7 52.07 0)
 			(effects
@@
 	)
 	(symbol
-		(lib_id "power:+5V")
-		(at 162.56 50.8 0)
+		(lib_id "power:+12V")
+		(at 215.9 48.26 0)
 		(unit 1)
 		(exclude_from_sim no)
@@
 		(on_board yes)
 		(dnp no)
-		(property "Reference" "#PWR038"
-			(at 162.56 54.61 0)
-			(effects
-				(font
-					(size 1.27 1.27)
-				)
-				(hide yes)
-			)
-		)
-		(property "Value" "+5V"
-			(at 165.862 49.022 0)
-			(effects
-				(font
-					(size 1.27 1.27)
+		(property "Reference" "#PWR107"
+			(at 215.9 52.07 0)
+			(effects
+				(font
+					(size 1.27 1.27)
+				)
+				(hide yes)
+			)
+		)
+		(property "Value" "+5V_MCU"
+			(at 215.9 44.196 0)
+			(effects
+				(font
+					(size 0.635 0.635)
 				)
 			)
 		)
 		(property "Footprint" ""
-			(at 162.56 50.8 0)
+			(at 215.9 48.26 0)
 			(effects
 				(font
@@
 		)
 		(property "Datasheet" ""
-			(at 162.56 50.8 0)
-			(effects
-				(font
-					(size 1.27 1.27)
-				)
-				(hide yes)
-			)
-		)
-		(property "Description" "Power symbol creates a global label with name \"+5V\""
-			(at 162.56 50.8 0)
+			(at 215.9 48.26 0)
+			(effects
+				(font
+					(size 1.27 1.27)
+				)
+				(hide yes)
+			)
+		)
+		(property "Description" ""
+			(at 215.9 48.26 0)
 			(effects
 				(font
@@
 			(project "steering_pcb"
 				(path "/27c2abcd-4c9d-416a-9e0c-4ab4decfd0fd/3158a1dc-35f2-49d2-93b5-e8517c53d7ab"
-					(reference "#PWR038")
+					(reference "#PWR107")
 					(unit 1)
 				)
@@
 		(in_bom no)
 		(on_board yes)
-		(dnp no)
+		(dnp yes)
 		(fields_autoplaced yes)
 		(property "Reference" "JP1"
@@
 		(property "Rating" ""
 			(at 33.02 119.38 0)
+			(effects
+				(font
+					(size 1.27 1.27)
+				)
+				(hide yes)
+			)
+		)
+		(property "Note" "I2C address pin"
+			(at 33.02 119.38 90)
 			(effects
 				(font
@@
 			)
 		)
-		(property "Datasheet" "~"
+		(property "Datasheet" "https://jlcpcb.com/partdetail/C25531"
 			(at 215.9 52.07 0)
 			(effects
@@
 			)
 		)
-		(property "Description" "Resistor, small symbol"
+		(property "Description" "0402WGJ0103TCE"
 			(at 215.9 52.07 0)
 			(effects
@@
 		)
 		(property "Rating" ""
+			(at 215.9 52.07 0)
+			(effects
+				(font
+					(size 1.27 1.27)
+				)
+				(hide yes)
+			)
+		)
+		(property "Note" "basic"
 			(at 215.9 52.07 0)
 			(effects
@@
 			)
 		)
-		(property "Datasheet" "https://www.lcsc.com/datasheet/lcsc_datasheet_2205311845_UNI-ROYAL-Uniroyal-Elec-0402WGJ0103TCE_C25531.pdf"
+		(property "Datasheet" "https://jlcpcb.com/partdetail/C25531"
 			(at 33.02 129.54 0)
 			(effects
@@
 			)
 		)
-		(property "Description" "Resistor, small symbol"
+		(property "Description" "0402WGJ0103TCE"
 			(at 33.02 129.54 0)
 			(effects
@@
 		)
 		(property "Rating" ""
+			(at 33.02 129.54 0)
+			(effects
+				(font
+					(size 1.27 1.27)
+				)
+				(hide yes)
+			)
+		)
+		(property "Note" "basic"
 			(at 33.02 129.54 0)
 			(effects
@@
 		(in_bom no)
 		(on_board yes)
-		(dnp no)
+		(dnp yes)
 		(fields_autoplaced yes)
 		(property "Reference" "JP6"
@@
 			(effects
 				(font
+					(size 1.27 1.27)
+				)
+				(hide yes)
+			)
+		)
+		(property "Note" "Gyroscope power solder jumper"
+			(at 91.44 41.91 90)
+			(effects
+				(font

Commit message: board update
Parts:
- removed Q1, Q6: BSS138BKS, PCM_Package_TO_SOT_SMD_AKL:SOT-363_SC-70-6, symbol PCM_Transistor_MOSFET_AKL:BSS138BKS
- added Q1: 2N7002DW, PCM_Package_TO_SOT_SMD_AKL:SOT-363_SC-70-6, symbol PCM_Transistor_MOSFET_AKL:2N7002DW
- R10, R12, R13, R8, R9: Product (none) -> 0402WGJ0103TCE
- TP_SCL3v1, TP_SDA3v1: now not fitted
- U5: Note (none) -> no
Connections:
- net MCU_SCL: now also Q1.6 (D1)
- net MCU_SDA: now also Q1.3 (D2)
- net SCL_3V: now also Q1.1 (S1)
- net SDA_3V: now also Q1.4 (S2)
- net at JP6.1 (A), R12.1, R9.1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: now also Q1.2 (G1), Q1.5 (G2)

Commit message: Rename folders for consistency
Parts:
- R10, R12, R13, R8, R9: value 10k -> 10kΩ
- U5: value ISM330DHCX -> ~; Product (none) -> C2943126
Changed lines of the file:
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@@
 (kicad_sch
-	(version 20231120)
+	(version 20250114)
 	(generator "eeschema")
-	(generator_version "8.0")
+	(generator_version "9.0")
 	(paper "A4")
 	(title_block
@@
 		(company "DTU ROAST")
 	)
+	(rectangle
+		(start 124.46 34.29)
+		(end 229.87 68.58)
+		(stroke
+			(width 0)
+			(type default)
+		)
+		(fill
+			(type none)
+		)
+	)
+	(rectangle
+		(start 24.13 95.25)
+		(end 77.47 142.24)
+		(stroke
+			(width 0)
+			(type default)
+		)
+		(fill
+			(type none)
+		)
+	)
+	(rectangle
+		(start 62.992 25.4)
+		(end 122.682 91.44)
+		(stroke
+			(width 0)
+			(type default)
+		)
+		(fill
+			(type none)
+		)
+	)
+	(text "Reference:\nhttps://learn.adafruit.com/lsm6dsox-and-ism330dhc-6-dof-imu?view=all\ncredits to adafruit"
+		(exclude_from_sim no)
+		(at 178.562 170.942 0)
+		(effects
+			(font
+				(size 1.3 1.3)
+			)
+			(justify left)
+		)
+	)
+	(text "Gyroscope Chip"
+		(exclude_from_sim no)
+		(at 72.39 28.956 0)
+		(effects
+			(font
+				(size 2 2)
+				(thickness 0.4)
+				(bold yes)
+			)
+			(justify left)
+		)
+	)
+	(text "Alternative power supply, but currently power is delivered by the 3v3 directly from the arduino MCU"
+		(exclude_from_sim no)
+		(at 224.028 125.476 0)
+		(effects
+			(font
+				(size 1.27 1.27)
+			)
+		)
+	)
+	(text "I2C Address pin. Pulling this pin high or bridging\nthe solder jumper on the back will change the I2C\naddress from 0x6A to 0x6B"
+		(exclude_from_sim no)
+		(at 25.654 101.6 0)
+		(effects
+			(font
+				(size 1.27 1.27)
+			)
+			(justify left)
+		)
+	)
+	(text "i2c pullup and shift"
+		(exclude_from_sim no)
+		(at 126.492 38.1 0)
+		(effects
+			(font
+				(size 2 2)
+				(thickness 0.4)
+				(bold yes)
+			)
+			(justify left)
+		)
+	)
 	(junction
 		(at 139.7 45.72)
@@
 			(width 0)
 			(type default)
-		)
-	)
-	(rectangle
-		(start 124.46 34.29)
-		(end 229.87 68.58)
-		(stroke
-			(width 0)
-			(type default)
-		)
-		(fill
-			(type none)
-		)
-	)
-	(rectangle
-		(start 24.13 95.25)
-		(end 77.47 142.24)
-		(stroke
-			(width 0)
-			(type default)
-		)
-		(fill
-			(type none)
-		)
-	)
-	(rectangle
-		(start 62.992 25.4)
-		(end 122.682 91.44)
-		(stroke
-			(width 0)
-			(type default)
-		)
-		(fill
-			(type none)
 		)
 	)
@@
 		)
 	)
-	(text "Reference:\nhttps://learn.adafruit.com/lsm6dsox-and-ism330dhc-6-dof-imu?view=all\ncredits to adafruit"
-		(exclude_from_sim no)
-		(at 178.562 170.942 0)
-		(effects
-			(font
-				(size 1.3 1.3)
-			)
-			(justify left)
-		)
-	)
-	(text "Gyroscope Chip"
-		(exclude_from_sim no)
-		(at 72.39 28.956 0)
-		(effects
-			(font
-				(size 2 2)
-				(thickness 0.4)
-				(bold yes)
-			)
-			(justify left)
-		)
-	)
-	(text "Alternative power supply, but currently power is delivered by the 3v3 directly from the arduino MCU"
-		(exclude_from_sim no)
-		(at 224.028 125.476 0)
-		(effects
-			(font
-				(size 1.27 1.27)
-			)
-		)
-	)
-	(text "I2C Address pin. Pulling this pin high or bridging\nthe solder jumper on the back will change the I2C\naddress from 0x6A to 0x6B"
-		(exclude_from_sim no)
-		(at 25.654 101.6 0)
-		(effects
-			(font
-				(size 1.27 1.27)
-			)
-			(justify left)
-		)
-	)
-	(text "i2c pullup and shift"
-		(exclude_from_sim no)
-		(at 126.492 38.1 0)
-		(effects
-			(font
-				(size 2 2)
-				(thickness 0.4)
-				(bold yes)
-			)
-			(justify left)
-		)
-	)
 	(global_label "SCL_3V"
 		(shape input)
@@
 			)
 		)
-		(property "Value" "10k"
+		(property "Value" "10kΩ"
 			(at 165.1 55.8799 0)
 			(effects
@@
 			)
 		)
-		(property "Value" "10k"
+		(property "Value" "10kΩ"
 			(at 195.58 53.3399 0)
 			(effects
@@
 			)
 		)
-		(property "Value" "10k"
+		(property "Value" "10kΩ"
 			(at 142.24 53.3399 0)
 			(effects
@@
 			)
 		)
-		(property "Value" "10k"
+		(property "Value" "10kΩ"
 			(at 218.44 53.3399 0)
 			(effects
@@
 			)
 		)
-		(property "Value" "ISM330DHCX"
+		(property "Value" "~"
 			(at 96.1741 87.63 0)
 			(effects
@@
 		)
 		(property "Note" "no"
+			(at 93.98 67.31 0)
+			(effects
+				(font
+					(size 1.27 1.27)
+				)
+				(hide yes)
+			)
+		)
+		(property "Product" "C2943126"
 			(at 93.98 67.31 0)
 			(effects
@@
 			)
 		)
-		(property "Value" "10k"
+		(property "Value" "10kΩ"
 			(at 34.29 130.556 0)
 			(effects
