File: Parts/steering_wheel_2025/steering_pcb/steering_pcb.kicad_pcb (KiCad board)
At the start: 2 copper layers, 102 x 102 mm, 195 parts, among them J0 Quick_connector, J1 Button 1 molex-µfit connector, J10 Button 1 molex-µfit connector, J11 Button 1 molex-µfit connector, J12 Button 1 molex-µfit connector, J13 PINHD_1x1_Male, J14 Conn_01x04_Pin, J15 CAN pin header, J16 Conn_01x01_Pin, J2 Button 1 molex-µfit connector, J3 Button 1 molex-µfit connector, J4 Button 1 molex-µfit connector, J5 Button 1 molex-µfit connector, J6 Button 1 molex-µfit connector, J7 Button 1 molex-µfit connector, J8 Button 1 molex-µfit connector, J9 Button 1 molex-µfit connector, Q1 BSS138BKS, Q10 2N7002DW, Q11 2N7002DW, Q12 2N7002DW, Q13 2N7002DW, Q14 2N7002DW, Q15 2N7002DW, Q16 2N7002DW, Q17 2N7002DW, Q18 2N7002DW, Q19 2N7002DW, Q2 2N7002DW, Q20 2N7002DW, Q21 2N7002DW, Q3 2N7002DW, Q4 BS170, Q5 2N7002DW, Q6 BSS138BKS, Q7 2N7002DW, Q8 2N7002DW, Q9 2N7002DW, SW1 Push_Button, U1 MCP2515-xSO, U2 TPS5430DDA, U3 TPS5430DDA, U5 ISM330DHCX, U6 TJA1051T-3, Y1 16MHz

Commit message: Dashboard electron
Parts:
- added F1: 176-9047, ROAST:Fuseholder_Clip-5x20mm_Littelfuse_520_Inline_P21.50x5.80mm_D1.30mm_Horizontal, B.Cu at (63.5, 132.7)
- moved D16 217.1 mm to (-12.2, 84.5)
- moved J0 216.5 mm to (-6.57, 106.6)
- moved R2 213.1 mm to (-2.13, 93.9), turned to -90 degrees
- moved U6 212.5 mm to (-5.46, 89.5)
- moved C12 212.5 mm to (-5.74, 97.4)
- moved C14 212.5 mm to (-9.63, 95.5)
- moved C15 212.5 mm to (-2.70, 98.4)
- moved D14 212.5 mm to (-5.68, 100.3)
- moved JP4 212.5 mm to (-4.54, 95.2)
- moved R26 212.5 mm to (-7.17, 94.9)
- moved C2 164.1 mm to (67.1, 59.2), turned to -90 degrees
- moved Y1 157.1 mm to (70.7, 59.3), turned to -90 degrees
- moved C1 151.4 mm to (73.7, 59.3), turned to 90 degrees
- moved C6 147.8 mm to (65.6, 127.7)
- moved C9 147.8 mm to (81.6, 132.8)
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Connections:
- J0 pad 3: +12V -> Net-(F1-Pad2)
Routing:
- net Net-(JP5-A): track 39.2 -> 8.36 mm
- net Net-(JP3-A): track 20.8 -> 0.00 mm
- net Net-(U1-TXCAN): track 19.4 -> 0.00 mm
- net Net-(A1-D0/RX0): track 17.1 -> 0.00 mm
- net Net-(U1-RXCAN): track 15.7 -> 0.00 mm
- net MCU_CLK: track 13.6 -> 0.00 mm
- net MCU_MISO: track 13.6 -> 0.00 mm
- net MCU_MOSI: track 13.1 -> 0.00 mm
- net ~{INT}: track 11.8 -> 0.00 mm
- net MCU_5V: track 10.1 -> 0.00 mm
- net CAN_L: track 23.8 -> 13.8 mm
- net MCU_GND: track 9.59 -> 0.00 mm
- net CAN_H: track 25.4 -> 18.7 mm
- net +3.3V: track 104.5 -> 98.0 mm, vias 5 -> 2
- net Net-(D16-Pad2): track 2.14 -> 0.00 mm
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