File: Parts/steering_wheel_2025/steering_pcb/steering_pcb.kicad_sch (KiCad schematic)
At the start: 34 parts, among them J0 Quick_connector, J14 Conn_01x04_Pin, J15 CAN pin header, J16 Conn_01x01_Pin, SW1 Push_Button, U2 TPS5430DDA, U3 TPS5430DDA

Commit message: Dashboard electron
Parts:
- added F1: 176-9047, ROAST:Fuseholder_Clip-5x20mm_Littelfuse_520_Inline_P21.50x5.80mm_D1.30mm_Horizontal, symbol Device:Fuse
- C10, C11, C16, C3, C6, C8: value GRM32ER61E226KE15L -> 22uF
- C17: value 10TPB220ML -> 220uF
- R5: value FRC0402F2101TS -> 2.1k
Connections:
- net +12V: now also F1.1; no longer J0.3
- new net: F1.2, J0.3
Other:
- note added: "A small switch mode buck converter that can supply up to 3A."
- note removed: "An small switch mode buck converter that can supply up to 3A."
- moved on the sheet: C11, C16, C17, C6, D13, J0, L3, R4, R5
