File: Parts/steering_wheel_2025/steering_pcb/LED.kicad_sch (KiCad schematic)
At the start: 3 parts, among them J13 PINHD_1x1_Male, Q4 BS170

Commit message: Error fixing with kicad_dru, and silkscreeen updates. TO-DO: BOM to basic
Parts:
- J13, JP8: now not fitted
Other:
- note added: "For connecting external LEDs, that dim with buttons"
Changed lines of the file:
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@@
 		)
 	)
+	(rectangle
+		(start 57.15 13.97)
+		(end 105.41 48.26)
+		(stroke
+			(width 0)
+			(type default)
+		)
+		(fill
+			(type none)
+		)
+	)
 	(image
 		(at 50.8 106.68)
@@
 		)
 	)
+	(text "For connecting external LEDs,\nthat dim with buttons"
+		(exclude_from_sim no)
+		(at 81.28 45.72 0)
+		(effects
+			(font
+				(size 1 1)
+			)
+			(justify left)
+		)
+	)
 	(text "Suitable current-limiting resistor\n\nBy burning LEDs\n\nBlue and Green works fine at 3.3v\nRed works fine at 3.3V with 47Ω resistor\n\nFor red LED\n(3v-2.3v)/15mA = 47Ω\n(5v-2.3v)/15mA = 180Ω\n(7v-2.3v)/15mA = 313Ω\n\nFor green and blue at higher voltages\n(5v-3.3v)/15mA = 113Ω\n(7v-3.3v)/15mA = 246Ω"
 		(exclude_from_sim no)
@@
 		(in_bom yes)
 		(on_board yes)
-		(dnp no)
+		(dnp yes)
 		(property "Reference" "J13"
 			(at 85.09 42.672 0)
@@
 		(in_bom no)
 		(on_board yes)
-		(dnp no)
+		(dnp yes)
 		(property "Reference" "JP8"
 			(at 74.422 42.418 0)

Commit message: board update
Parts:
- Q4: footprint PCM_Package_TO_SOT_THT_AKL:TO-92_Inline_Wide_DGS -> Package_TO_SOT_THT:TO-92_Inline_Wide; JLCPCB C2998067 -> C111691; Note (none) -> maybe?? no; Product (none) -> BS170
Changed lines of the file:
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@@
 			)
 		)
-		(property "Footprint" "PCM_Package_TO_SOT_THT_AKL:TO-92_Inline_Wide_DGS"
+		(property "Footprint" "Package_TO_SOT_THT:TO-92_Inline_Wide"
 			(at 73.66 24.13 0)
 			(effects
@@
 			)
 		)
-		(property "JLCPCB" "C2998067"
+		(property "JLCPCB" "C111691"
 			(at 78.74 26.67 0)
 			(effects
@@
 			(at 78.74 26.67 0)
 			(effects
+				(font
+					(size 1.27 1.27)
+				)
+				(hide yes)
+			)
+		)
+		(property "Product" "BS170"
+			(at 78.74 26.67 0)
+			(effects
+				(font
+					(size 1.27 1.27)
+				)
+				(hide yes)
+			)
+		)
+		(property "Note" "maybe?? no"
+			(at 78.74 26.67 0)
+			(effects
