File: Parts/steering_wheel_2025/steering_pcb/LED.kicad_sch (KiCad schematic)
At the start: 3 parts, among them J13 PINHD_1x1_Male, Q4 BS170

Commit message: Rename folders for consistency
Changed lines of the file:
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@@
 (kicad_sch
-	(version 20231120)
+	(version 20250114)
 	(generator "eeschema")
-	(generator_version "8.0")
+	(generator_version "9.0")
 	(paper "A4")
 	(title_block
@@
 		(company "DTU ROAST")
 	)
+	(rectangle
+		(start 57.15 13.97)
+		(end 105.41 48.26)
+		(stroke
+			(width 0)
+			(type default)
+		)
+		(fill
+			(type none)
+		)
+	)
+	(text "Transistor for turning on LEDs\nThe 2N7002 requires a Vgs of around 2-4V to turn\non fully\n\nBZX84C3V3TS-7-F is a zener diode that blocks for voltages below 3.3v.\n"
+		(exclude_from_sim no)
+		(at 14.478 120.142 0)
+		(effects
+			(font
+				(size 1.27 1.27)
+			)
+			(justify left top)
+		)
+	)
+	(text "Using other buttons than x_0, the 7V connection as HIGH is neccessary.\nFor x_0, one can get away with a 5V HIGH connection."
+		(exclude_from_sim no)
+		(at 14.478 143.51 0)
+		(effects
+			(font
+				(size 1.27 1.27)
+			)
+			(justify left)
+		)
+	)
+	(text "For connecting external LEDs,\nthat dim with buttons"
+		(exclude_from_sim no)
+		(at 81.28 45.72 0)
+		(effects
+			(font
+				(size 1 1)
+			)
+			(justify left)
+		)
+	)
+	(text "Suitable current-limiting resistor\n\nBy burning LEDs\n\nBlue and Green works fine at 3.3v\nRed works fine at 3.3V with 47Ω resistor\n\nFor red LED\n(3v-2.3v)/15mA = 47Ω\n(5v-2.3v)/15mA = 180Ω\n(7v-2.3v)/15mA = 313Ω\n\nFor green and blue at higher voltages\n(5v-3.3v)/15mA = 113Ω\n(7v-3.3v)/15mA = 246Ω"
+		(exclude_from_sim no)
+		(at 14.732 41.148 0)
+		(effects
+			(font
+				(size 1.27 1.27)
+			)
+			(justify left top)
+		)
+	)
 	(wire
 		(pts
@@
 		)
 	)
-	(rectangle
-		(start 57.15 13.97)
-		(end 105.41 48.26)
-		(stroke
-			(width 0)
-			(type default)
-		)
-		(fill
-			(type none)
-		)
-	)
 	(image
 		(at 50.8 106.68)
@@
 		)
 	)
-	(text "Transistor for turning on LEDs\nThe 2N7002 requires a Vgs of around 2-4V to turn\non fully\n\nBZX84C3V3TS-7-F is a zener diode that blocks for voltages below 3.3v.\n"
-		(exclude_from_sim no)
-		(at 14.478 120.142 0)
-		(effects
-			(font
-				(size 1.27 1.27)
-			)
-			(justify left top)
-		)
-	)
-	(text "Using other buttons than x_0, the 7V connection as HIGH is neccessary.\nFor x_0, one can get away with a 5V HIGH connection."
-		(exclude_from_sim no)
-		(at 14.478 143.51 0)
-		(effects
-			(font
-				(size 1.27 1.27)
-			)
-			(justify left)
-		)
-	)
-	(text "For connecting external LEDs,\nthat dim with buttons"
-		(exclude_from_sim no)
-		(at 81.28 45.72 0)
-		(effects
-			(font
-				(size 1 1)
-			)
-			(justify left)
-		)
-	)
-	(text "Suitable current-limiting resistor\n\nBy burning LEDs\n\nBlue and Green works fine at 3.3v\nRed works fine at 3.3V with 47Ω resistor\n\nFor red LED\n(3v-2.3v)/15mA = 47Ω\n(5v-2.3v)/15mA = 180Ω\n(7v-2.3v)/15mA = 313Ω\n\nFor green and blue at higher voltages\n(5v-3.3v)/15mA = 113Ω\n(7v-3.3v)/15mA = 246Ω"
-		(exclude_from_sim no)
-		(at 14.732 41.148 0)
-		(effects
-			(font
-				(size 1.27 1.27)
-			)
-			(justify left top)
-		)
-	)
 	(global_label "button10_1"
 		(shape input)
@@
 		(at 124.46 34.29)
 		(size 33.02 17.78)
+		(exclude_from_sim no)
+		(in_bom yes)
+		(on_board yes)
+		(dnp no)
 		(fields_autoplaced yes)
 		(stroke
@@
 		(at 185.42 85.09)
 		(size 33.02 17.78)
+		(exclude_from_sim no)
+		(in_bom yes)
+		(on_board yes)
+		(dnp no)
 		(fields_autoplaced yes)
 		(stroke
@@
 		(at 124.46 85.09)
 		(size 33.02 17.78)
+		(exclude_from_sim no)
+		(in_bom yes)
+		(on_board yes)
+		(dnp no)
 		(fields_autoplaced yes)
 		(stroke
@@
 		(at 185.42 34.29)
 		(size 33.02 17.78)
+		(exclude_from_sim no)
+		(in_bom yes)
+		(on_board yes)
+		(dnp no)
 		(fields_autoplaced yes)
 		(stroke
@@
 		(at 124.46 59.69)
 		(size 33.02 17.78)
+		(exclude_from_sim no)
+		(in_bom yes)
+		(on_board yes)
+		(dnp no)
 		(fields_autoplaced yes)
 		(stroke
@@
 		(at 185.42 59.69)
 		(size 33.02 17.78)
+		(exclude_from_sim no)
+		(in_bom yes)
+		(on_board yes)
+		(dnp no)
 		(fields_autoplaced yes)
 		(stroke
